File: VoidHHKB-Hotswap.kicad_pcb (KiCad board)
At the start: 2 copper layers, 286.4 x 96.1 mm, 152 parts, among them J2 TC2030_SWD, U1 XC6206P332MR, U2 STM32F072CBT6

Commit message: Removed switch sockets that can't be used due to plate limitations.
Parts:
- removed MX61: MX_SW_HS, PCM_marbastlib-mx:SW_MX_HS_CPG151101S11_1u
- removed MX62: MX_SW_HS, PCM_marbastlib-mx:SW_MX_HS_CPG151101S11_1.75u_STP_1.25
- moved D31 9.37 mm to (48.2, 76.5), turned to 90 degrees
- turned MX30 to 180 degrees
Routing:
- net Net-(D31-A): track 37.9 -> 8.93 mm
- net PB12: track 336.8 -> 322.7 mm, vias 7 -> 6
- net Net-(D59-A): track 15.6 -> 3.61 mm
- net NRST: track 40.2 -> 43.2 mm
- net PB2: track 289.7 -> 286.7 mm
- net PA5: track 229.0 -> 227.0 mm
- net GND: track 66.3 -> 66.9 mm, vias 7 -> 16

Commit message: Added Solder PCB
Other:
- board text added: "VoidHHKB-Hotswap"
- board text added: "ver. ${CURRENT_DATE}"
Changed lines of the file:
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@@
 		(fp_arc
 			(start 9.03125 8.000001)
-			(mid 8.677693 7.853543)
+			(mid 8.677729 7.853537)
 			(end 8.53125 7.500001)
 			(stroke
@@
 		(fp_arc
 			(start 14.780039 -5.999999)
-			(mid 15.133602 -5.853545)
+			(mid 15.133567 -5.853539)
 			(end 15.280039 -5.499999)
 			(stroke
@@
 		(fp_arc
 			(start 15.28125 7.500001)
-			(mid 15.1348 7.853536)
+			(mid 15.134806 7.853571)
 			(end 14.78125 8.000001)
 			(stroke
@@
 		(fp_arc
 			(start 9.03125 8.000001)
-			(mid 8.677693 7.853543)
+			(mid 8.677729 7.853537)
 			(end 8.53125 7.500001)
 			(stroke
@@
 		(fp_arc
 			(start 14.780039 -5.999999)
-			(mid 15.133602 -5.853545)
+			(mid 15.133567 -5.853539)
 			(end 15.280039 -5.499999)
 			(stroke
@@
 		(fp_arc
 			(start 15.28125 7.500001)
-			(mid 15.1348 7.853536)
+			(mid 15.134806 7.853571)
 			(end 14.78125 8.000001)
 			(stroke
@@
 		(descr "Footprint for Cherry MX style switches with Kailh hotswap socket")
 		(property "Reference" "MX30"
-			(at -4.25 1.75 360)
+			(at -4.25 1.75 0)
 			(layer "B.SilkS")
 			(effects
@@
 		)
 		(property "Value" "MX_SW_HS"
-			(at 0 0 360)
+			(at 0 0 0)
 			(layer "B.Fab")
 			(effects
@@
 		)
 		(property "Footprint" "PCM_marbastlib-mx:SW_MX_HS_CPG151101S11_1.75u"
-			(at 0 0 360)
+			(at 0 0 0)
 			(layer "B.Fab")
 			(hide yes)
@@
 		)
 		(property "Datasheet" ""
-			(at 0 0 360)
+			(at 0 0 0)
 			(layer "B.Fab")
 			(hide yes)
@@
 		)
 		(property "Description" "Push button switch, normally open, two pins, 45° tilted, Kailh CPG151101S11 for Cherry MX style switches"
-			(at 0 0 360)
+			(at 0 0 0)
 			(layer "B.Fab")
 			(hide yes)
@@
 		)
 		(fp_text user "${REFERENCE}"
-			(at 0.5 4.5 360)
+			(at 0.5 4.5 0)
 			(layer "B.Fab")
 			(effects
@@
 		)
 	)
+	(gr_rect
+		(start 117.0629 104.34455)
+		(end 148.10435 111.4883)
+		(stroke
+			(width 0.5)
+			(type default)
+		)
+		(fill none)
+		(layer "B.SilkS")
+	)
 	(gr_line
 		(start 310.462509 26.78967)
@@
 		(layer "Edge.Cuts")
 	)
+	(gr_text "VoidHHKB-Hotswap"
+		(at 132.7742 108.3133 0)
+		(layer "B.SilkS")
+		(effects
+			(font
+				(size 2 2)
+				(thickness 0.5)
+				(bold yes)
+			)
+			(justify bottom mirror)
+		)
+	)
+	(gr_text "ver. ${CURRENT_DATE}"
+		(at 132.7742 109.10705 0)
+		(layer "B.SilkS")
+		(effects
+			(font
+				(size 1 1)
+				(thickness 0.25)
+				(bold yes)
+			)
+			(justify top mirror)
+		)
+	)
 	(segment
