File: VoidHHKB-Solder/VoidHHKB-Solder.kicad_pcb (KiCad board)
At the start: 2 copper layers, 286.4 x 96.1 mm, 163 parts, among them J2 TC2030_SWD, U1 XC6206P332MR, U2 STM32F072CBT6

Commit message: Updated Solder PCB. Fix designators and add labels to silk screen.
Parts:
- removed the G*** at (36.1, 109.4)
- removed the G*** at (295.6, 109.3)
- removed the G*** at (187.8, 109.2)
- added G***: LOGO, LOGO, F.Cu at (28.4, 101.8)
- added G***: LOGO, LOGO, F.Cu at (287.8, 101.7)
- added G***: LOGO, LOGO, F.Cu at (180.0, 101.6)
- MX1: value MX_SW_HS -> Esc
- MX10: value MX_SW_HS -> 9
- MX11: value MX_SW_HS -> 10
- MX12: value MX_SW_HS -> -
- MX13: value MX_SW_HS -> =
- MX14: value MX_SW_HS -> \
- MX15: value MX_SW_HS -> `
- MX16: value MX_SW_HS -> Full Backspace
- MX17: value MX_SW_HS -> Tab; footprint PCM_marbastlib-mx:SW_MX_1u -> PCM_marbastlib-mx:SW_MX_1.5u
- MX18: value MX_SW_HS -> Q
- MX19: value MX_SW_HS -> W
- MX2: value MX_SW_HS -> 1
- MX20: value MX_SW_HS -> E
- MX21: value MX_SW_HS -> R
- MX22: value MX_SW_HS -> T
- MX23: value MX_SW_HS -> Y
- MX24: value MX_SW_HS -> U
- MX25: value MX_SW_HS -> I
- MX26: value MX_SW_HS -> O
- MX27: value MX_SW_HS -> P
- MX28: value MX_SW_HS -> [
- MX29: value MX_SW_HS -> ]
- MX3: value MX_SW_HS -> 2
- MX30: value MX_SW_HS -> Backspace; footprint PCM_marbastlib-mx:SW_MX_1.75u_STP_1.25 -> PCM_marbastlib-mx:SW_MX_1.5u
- MX31: value MX_SW_HS -> Stepped Caps; footprint PCM_marbastlib-mx:SW_MX_1u -> PCM_marbastlib-mx:SW_MX_1.75u_STP_1.25
- MX32: value MX_SW_HS -> A
- MX33: value MX_SW_HS -> S
- MX34: value MX_SW_HS -> D
- MX35: value MX_SW_HS -> F
- MX36: value MX_SW_HS -> G
- MX37: value MX_SW_HS -> H
- MX38: value MX_SW_HS -> J
- MX39: value MX_SW_HS -> K
- MX4: value MX_SW_HS -> 3
- MX40: value MX_SW_HS -> L
- MX41: value MX_SW_HS -> ;
- MX42: value MX_SW_HS -> '
- MX43, MX48: value MX_SW_HS -> NUHS
- MX44: value MX_SW_HS -> ANSI Enter
- MX45: value MX_SW_HS -> Caps; footprint PCM_marbastlib-mx:SW_MX_1u -> PCM_marbastlib-mx:SW_MX_1.75u
- MX46: value MX_SW_HS -> ISO Enter
- MX47: value MX_SW_HS -> LShift
- MX49: value MX_SW_HS -> Z
- MX5: value MX_SW_HS -> 4
- MX50: value MX_SW_HS -> X
- MX51: value MX_SW_HS -> C
- MX52: value MX_SW_HS -> V
- MX53: value MX_SW_HS -> B
- MX54: value MX_SW_HS -> N
- MX55: value MX_SW_HS -> M
- MX56: value MX_SW_HS -> ,
- MX57: value MX_SW_HS -> .
- MX58: value MX_SW_HS -> /
- MX59: value MX_SW_HS -> RShift 1.75u; footprint PCM_marbastlib-mx:SW_MX_1u -> PCM_marbastlib-mx:SW_MX_1.75u
- MX6: value MX_SW_HS -> 5
- MX60: value MX_SW_HS -> fn
- MX61: value MX_SW_HS -> LShift 1.25u; footprint PCM_marbastlib-mx:SW_MX_1u -> PCM_marbastlib-mx:SW_MX_1.25u
- MX62: value MX_SW_HS -> RShift 2.75u; footprint PCM_marbastlib-mx:SW_MX_1.75u -> PCM_marbastlib-mx:SW_MX_1u
- MX63, MX67: value MX_SW_HS -> Alt
- MX64, MX66: value MX_SW_HS -> Super; footprint PCM_marbastlib-mx:SW_MX_1u -> PCM_marbastlib-mx:SW_MX_1.5u
- MX65: value NUHS -> Spacebar
- MX68: value MX_SW_HS -> Off Center Spacebar
- MX7: value MX_SW_HS -> 6
- MX8: value MX_SW_HS -> 7
- MX9: value MX_SW_HS -> 8
- S1: value 2.25u ANSI Enter -> 2u Backspace; footprint PCM_marbastlib-mx:STAB_MX_2.25u -> PCM_marbastlib-mx:STAB_MX_2u
- S2: value 2.25 LShift -> 2.25u ANSI Enter
- S3: value 6u Spacebar -> ISO Enter; footprint PCM_marbastlib-mx:STAB_MX_6u_New -> PCM_marbastlib-mx:STAB_MX_ISO-ROT
- S4: value 2u Backspace -> 2.25 LShift; footprint PCM_marbastlib-mx:STAB_MX_2u -> PCM_marbastlib-mx:STAB_MX_2.25u
- S5: value ISO Enter -> 2.75 RShift; footprint PCM_marbastlib-mx:STAB_MX_ISO-ROT -> PCM_marbastlib-mx:STAB_MX_2.75u
- S6: value 2.75 RShift -> 6u Spacebar; footprint PCM_marbastlib-mx:STAB_MX_2.75u -> PCM_marbastlib-mx:STAB_MX_6u_New
- moved S4 257.8 mm to (38.1, 83.3)
- moved MX30 253.2 mm to (288.1, 45.2)
- moved MX63 246.1 mm to (54.8, 102.4)
- moved MX16 246.1 mm to (283.4, 26.2)
- moved D44 241.3 mm to (288.1, 68.9)
- moved S2 236.7 mm to (281.0, 64.3), turned to 180 degrees
- moved MX62 235.4 mm to (276.2, 83.3)
- moved MX43 224.8 mm to (269.1, 64.3)
- moved MX64 223.3 mm to (78.6, 102.4)
- moved MX67 211.6 mm to (245.3, 102.4)
- moved MX44 205.9 mm to (281.0, 64.3)
- moved D58 204.7 mm to (300.0, 88.1), turned to 90 degrees
- moved D57 202.4 mm to (273.8, 88.1), turned to 90 degrees
- moved D63 194.2 mm to (254.8, 95.3), turned to -90 degrees
- moved MX46 179.3 mm to (290.5, 54.8)
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Connections:
- D44 pad 1: PB1 -> PB2
- D57 pad 1: PB0 -> PB1
- D58 pad 1: PB0 -> PB1
- D62 pad 1: PB2 -> PB0
- D63 pad 1: PB1 -> PB0
- MX16 pad 1: PB12 -> PB3
- MX16 pad 2: Net-(D17-A) -> Net-(D15-A)
- MX17 pad 1: PA3 -> PB12
- MX17 pad 2: Net-(D18-A) -> Net-(D17-A)
- MX18 pad 1: PA4 -> PA3
- MX18 pad 2: Net-(D19-A) -> Net-(D18-A)
- MX19 pad 1: PB14 -> PA4
- MX19 pad 2: Net-(D20-A) -> Net-(D19-A)
- MX20 pad 1: PB15 -> PB14
- MX20 pad 2: Net-(D21-A) -> Net-(D20-A)
- MX21 pad 1: PA8 -> PB15
- MX21 pad 2: Net-(D22-A) -> Net-(D21-A)
- MX22 pad 1: PA5 -> PA8
- MX22 pad 2: Net-(D23-A) -> Net-(D22-A)
- MX23 pad 1: PA9 -> PA5
- MX23 pad 2: Net-(D24-A) -> Net-(D23-A)
- MX24 pad 1: PA10 -> PA9
- MX24 pad 2: Net-(D25-A) -> Net-(D24-A)
- MX25 pad 1: PA6 -> PA10
- MX25 pad 2: Net-(D26-A) -> Net-(D25-A)
- MX26 pad 1: PA7 -> PA6
- MX26 pad 2: Net-(D27-A) -> Net-(D26-A)
- MX27 pad 1: PA15 -> PA7
- MX27 pad 2: Net-(D28-A) -> Net-(D27-A)
- MX28 pad 1: PB3 -> PA15
- MX28 pad 2: Net-(D29-A) -> Net-(D28-A)
- MX29 pad 1: PB4 -> PB3
- MX29 pad 2: Net-(D30-A) -> Net-(D29-A)
- MX30 pad 1: PB12 -> PB4
- MX30 pad 2: Net-(D31-A) -> Net-(D30-A)
- MX31 pad 1: PA3 -> PB12
- MX31 pad 2: Net-(D32-A) -> Net-(D31-A)
- MX32 pad 1: PA4 -> PA3
- MX32 pad 2: Net-(D33-A) -> Net-(D32-A)
- MX33 pad 1: PB14 -> PA4
- MX33 pad 2: Net-(D34-A) -> Net-(D33-A)
- MX34 pad 1: PB15 -> PB14
- MX34 pad 2: Net-(D35-A) -> Net-(D34-A)
- MX35 pad 1: PA8 -> PB15
- MX35 pad 2: Net-(D36-A) -> Net-(D35-A)
- MX36 pad 1: PA5 -> PA8
- MX36 pad 2: Net-(D37-A) -> Net-(D36-A)
- MX37 pad 1: PA9 -> PA5
- MX37 pad 2: Net-(D38-A) -> Net-(D37-A)
- MX38 pad 1: PA10 -> PA9
- MX38 pad 2: Net-(D39-A) -> Net-(D38-A)
- MX39 pad 1: PA6 -> PA10
- MX39 pad 2: Net-(D40-A) -> Net-(D39-A)
- MX40 pad 1: PA7 -> PA6
- MX40 pad 2: Net-(D41-A) -> Net-(D40-A)
- MX41 pad 1: PA15 -> PA7
- MX41 pad 2: Net-(D42-A) -> Net-(D41-A)
- MX42 pad 1: PB4 -> PA15
- MX42 pad 2: Net-(D43-A) -> Net-(D42-A)
- MX43 pad 1: PB12 -> PB3
- MX43 pad 2: Net-(D44-A) -> Net-(D43-A)
- MX44 pad 1: PA3 -> PB4
- MX44 pad 2: Net-(D45-A) -> Net-(D44-A)
- MX45 pad 1: PA4 -> PB12
- MX45 pad 2: Net-(D46-A) -> Net-(D31-A)
- MX46 pad 1: PB14 -> PB4
- MX46 pad 2: Net-(D47-A) -> Net-(D44-A)
- MX47 pad 1: PB15 -> PB12
- MX47 pad 2: Net-(D48-A) -> Net-(D45-A)
- MX48 pad 1: PA8 -> PB13
- MX48 pad 2: Net-(D49-A) -> Net-(D46-A)
- MX49 pad 1: PA5 -> PA3
- MX49 pad 2: Net-(D50-A) -> Net-(D47-A)
- MX50 pad 1: PA9 -> PA4
- MX50 pad 2: Net-(D51-A) -> Net-(D48-A)
- MX51 pad 1: PA10 -> PB14
- MX51 pad 2: Net-(D52-A) -> Net-(D49-A)
- MX52 pad 1: PA6 -> PB15
- MX52 pad 2: Net-(D53-A) -> Net-(D50-A)
- MX53 pad 1: PA7 -> PA8
- MX53 pad 2: Net-(D54-A) -> Net-(D51-A)
- MX54 pad 1: PB3 -> PA5
- MX54 pad 2: Net-(D55-A) -> Net-(D52-A)
- MX55 pad 1: PB4 -> PA9
- MX55 pad 2: Net-(D56-A) -> Net-(D53-A)
- MX56 pad 1: PA3 -> PA10
- MX56 pad 2: Net-(D57-A) -> Net-(D54-A)
- MX57 pad 1: PA4 -> PA6
- MX57 pad 2: Net-(D58-A) -> Net-(D55-A)
- MX58 pad 1: PA5 -> PA7
- MX58 pad 2: Net-(D59-A) -> Net-(D56-A)
- MX59 pad 1: PA6 -> PB3
- MX59 pad 2: Net-(D60-A) -> Net-(D57-A)
- MX60 pad 1: PA7 -> PB4
- MX60 pad 2: Net-(D61-A) -> Net-(D58-A)
- MX61 pad 1: PA5 -> PB12
- MX61 pad 2: Net-(D59-A) -> Net-(D45-A)
- MX62 pad 1: PB12 -> PB3
- MX62 pad 2: Net-(D31-A) -> Net-(D57-A)
- MX63 pad 1: PB3 -> PA3
- MX63 pad 2: Net-(D15-A) -> Net-(D59-A)
- MX64 pad 1: PB4 -> PA4
- MX64 pad 2: Net-(D43-A) -> Net-(D60-A)
- MX65 pad 1: PB3 -> PA5
- MX65 pad 2: Net-(D62-A) -> Net-(D61-A)
- MX66 pad 1: PB13 -> PA6
- MX66 pad 2: Net-(D63-A) -> Net-(D62-A)
- MX67 pad 1: PB12 -> PA7
- MX67 pad 2: Net-(D44-A) -> Net-(D63-A)
- MX68 pad 1: PB3 -> PA5
- MX68 pad 2: Net-(D55-A) -> Net-(D61-A)
Routing:
- net Net-(D43-A): track 24.6 -> 7.72 mm
- net Net-(D57-A): track 7.14 -> 20.7 mm
- net Net-(D55-A): track 20.7 -> 10.1 mm
- net Net-(D59-A): track 16.7 -> 7.14 mm
- net Net-(D61-A): track 7.17 -> 16.7 mm
- net Net-(D45-A): track 10.1 -> 17.8 mm
- net Net-(D44-A): track 20.2 -> 24.6 mm
- net Net-(D58-A): track 7.12 -> 10.1 mm
- net Net-(D46-A): track 10.1 -> 8.31 mm
- net Net-(D63-A): track 8.31 -> 7.17 mm
- net Net-(D62-A): track 7.72 -> 7.18 mm
- net GND: vias 37 -> 36
- net VBUS: vias 4 -> 3
Other:
- board text added: "1.5u"
- board text added: "1u"
- board text added: "6u"
- board text added: "ANSI"
- board text added: "FULL"
- board text added: "ISO"
- board text added: "Off-Center"
- board text added: "REGULAR"
- board text added: "SPLIT"
- board text added: "STEPPED"
- board text added: "VoidHHKB-Solder"
- board text removed: "VoidHHKB-S"
